Commit message: Add files via upload

File: silver/description/ros2_control_silver.xacro (robot description, xacro)
@@ -12,5 +12,5 @@
                 <!--plugin>silver_dynamixel_hardware/SilverDynamixelHardware</plugin-->
                 <param name="usb_port">/dev/ttyUSB0</param>
-                <param name="baud_rate">57600</param>
+                <param name="baud_rate">1000000</param>
             </hardware>
         </xacro:unless>

File: silver/description/silver.xacro (robot description, xacro)
@@ -6,5 +6,5 @@
     <xacro:include filename="gazebo_control.xacro"/>
      <!-- Import Leg geometry Macro -->
-    <xacro:include filename="robot_leg.xacro"/>
+    <xacro:include filename="silver_leg.xacro"/>
      <!-- Import Leg control Macro -->
     <xacro:include filename="ros2_control_leg.xacro"/>
@@ -44,9 +44,9 @@
         </xacro:inertial_box>
     </link>
-    <xacro:leg suffix="0" reflect="1" Ox="0.35" Oy="0.3" Oz="-0.15"/>
-    <xacro:leg suffix="1" reflect="1" Ox="0.0" Oy="0.3" Oz="-0.15"/>
-    <xacro:leg suffix="2" reflect="1" Ox="-0.35" Oy="0.3" Oz="-0.15"/>
-    <xacro:leg suffix="3" reflect="-1" Ox="0.35" Oy="-0.3" Oz="-0.15"/>
-    <xacro:leg suffix="4" reflect="-1" Ox="0.0" Oy="-0.3" Oz="-0.15"/>
-    <xacro:leg suffix="5" reflect="-1" Ox="-0.35" Oy="-0.3" Oz="-0.15"/>
+    <xacro:leg suffix="0" reflect="1" side='right' Ox="0.275" Oy="-0.2" Oz="-0.15"/>
+    <xacro:leg suffix="1" reflect="1" side='right' Ox="0.0" Oy="-0.2" Oz="-0.15"/>
+    <xacro:leg suffix="2" reflect="-1" side='right' Ox="-0.275" Oy="-0.2" Oz="-0.15"/>
+    <xacro:leg suffix="3" reflect="-1" side='left' Ox="0.275" Oy="0.2" Oz="-0.15"/>
+    <xacro:leg suffix="4" reflect="-1" side='left' Ox="0.0" Oy="0.2" Oz="-0.15"/>
+    <xacro:leg suffix="5" reflect="1" side='left' Ox="-0.275" Oy="0.2" Oz="-0.15"/>
 </robot>

File: silver/description/silver_constants_new.xacro (robot description, xacro)
@@ -4,6 +4,6 @@
     <xacro:property name="body_link_mass" value="2.0" /> <!-- Kg -->
     <xacro:property name="body_link_height" value="1.0" /> <!-- m -->
-    <xacro:property name="body_link_x_dim" value="0.55" /> <!-- m -->
-    <xacro:property name="body_link_y_dim" value="0.4" /> <!-- m -->
+    <xacro:property name="body_link_x_dim" value="0.8" /> <!-- m -->
+    <xacro:property name="body_link_y_dim" value="0.6" /> <!-- m -->
     <xacro:property name="body_link_z_dim" value="0.3" /> <!-- m -->
     <xacro:property name="coxa_link_mass" value="0.5" /> <!-- Kg -->
@@ -12,5 +12,5 @@
     <xacro:property name="coxa_joint_Oz" value="0.0" /> <!-- m -->
     <xacro:property name="coxa_link_Ox" value="0.03" /> <!-- m -->
-    <xacro:property name="coxa_link_Oy" value="-0.05" /> <!-- m -->
+    <xacro:property name="coxa_link_Oy" value="0.05" /> <!-- m -->
     <xacro:property name="coxa_link_Oz" value="-0.05" /> <!-- m -->
     <xacro:property name="coxa_link_Ry" value="1.57" /> <!-- rad -->
@@ -18,24 +18,23 @@
     <xacro:property name="coxa_link_radius" value="0.05" /> <!-- m -->
     <xacro:property name="femur_link_mass" value="0.5" /> <!-- Kg -->
-    <xacro:property name="femur_joint_Ox" value="0.07" /> <!-- m -->
-    <xacro:property name="femur_joint_Oy" value="-0.05" /> <!-- m -->
+    <xacro:property name="femur_joint_Ox" value="0.09" /> <!-- m -->
+    <xacro:property name="femur_joint_Oy" value="0.05" /> <!-- m -->
     <xacro:property name="femur_joint_Oz" value="-0.05" /> <!-- m -->
-    <xacro:property name="femur_joint_Ry" value="-1.57" /> <!-- rad -->
-    <xacro:property name="femur_link_Ox" value="0.0" /> <!-- m -->
-    <xacro:property name="femur_link_Oy" value="-0.15" /> <!-- m -->
-    <xacro:property name="femur_link_Oz" value="-0.01" /> <!-- m -->
-    <xacro:property name="femur_link_dx" value="0.03" /> <!-- m -->
-    <xacro:property name="femur_link_dy" value="0.3" /> <!-- m -->
+    <xacro:property name="femur_joint_Ry" value="1.57" /> <!-- rad -->
+    <xacro:property name="femur_link_Ox" value="0.2" /> <!-- m -->
+    <xacro:property name="femur_link_Oy" value="0.05" /> <!-- m -->
+    <xacro:property name="femur_link_Oz" value="-0.05" /> <!-- m -->
+    <xacro:property name="femur_link_dx" value="0.4" /> <!-- m -->
+    <xacro:property name="femur_link_dy" value="0.03" /> <!-- m -->
     <xacro:property name="femur_link_dz" value="0.01" /> <!-- m -->
     <xacro:property name="tibia_link_mass" value="0.5" /> <!-- Kg -->
-    <xacro:property name="tibia_joint_Ox" value="0.0" /> <!-- m -->
-    <xacro:property name="tibia_joint_Oy" value="-0.3" /> <!-- m -->
-    <xacro:property name="tibia_joint_Oz" value="-0.01" /> <!-- m -->
-    <xacro:property name="tibia_link_Ry" value="3.14" /> <!-- rad -->
-    <xacro:property name="tibia_link_Ox" value="0.0" /> <!-- m -->
-    <xacro:property name="tibia_link_Oy" value="-0.15" /> <!-- m -->
+    <xacro:property name="tibia_joint_Ox" value="0.4" /> <!-- m -->
+    <xacro:property name="tibia_joint_Oy" value="0.0" /> <!-- m -->
+    <xacro:property name="tibia_joint_Oz" value="0.01" /> <!-- m -->
+    <xacro:property name="tibia_link_Ox" value="0.15" /> <!-- m -->
+    <xacro:property name="tibia_link_Oy" value="0.0" /> <!-- m -->
     <xacro:property name="tibia_link_Oz" value="0.0" /> <!-- m -->
-    <xacro:property name="tibia_link_dx" value="0.03" /> <!-- m -->
-    <xacro:property name="tibia_link_dy" value="-0.32" /> <!-- m -->
+    <xacro:property name="tibia_link_dx" value="0.3" /> <!-- m -->
+    <xacro:property name="tibia_link_dy" value="0.03" /> <!-- m -->
     <xacro:property name="tibia_link_dz" value="0.01" /> <!-- m -->
     <xacro:property name="foot_link_mass" value="0.1" /> <!-- Kg -->
