Commit message: Add files via upload

File: silver/description/gazebo_control.xacro (robot description, xacro)
@@ -1,12 +1,8 @@
 <?xml version="1.0"?>
 <robot xmlns:xacro="http://www.ros.org/wiki/xacro">
-    <!-- This file demonstrates the use of some <gazebo> tags -->
-    <!-- To include it add the following line -->
-    <!-- <xacro:include filename="example_gazebo.xacro" /> -->
-    <!-- Gazebo requires the use of plugins to interact with other systems such as ROS. -->
     <!-- ros_control plugin -->
     <gazebo>
       <plugin filename="libgazebo_ros2_control.so" name="gazebo_ros2_control">
-        <parameters>$(find silver)/config/my_controllers.yaml</parameters>
+        <parameters>$(find silver)/config/silver_controllers.yaml</parameters>
         <parameters>$(find silver)/config/gaz_ros2_control_use_sim.yaml</parameters>
       </plugin>
@@ -18,18 +14,93 @@
       <material>Gazebo/Blue</material>
     </gazebo>
-    <!-- Coxa Link -->
-    <gazebo reference="coxa_link">
+    <!-- Coxa Links -->
+    <gazebo reference="coxa_link_0">
       <mu1>0.2</mu1>
       <mu2>0.2</mu2>
       <material>Gazebo/Blue</material>
     </gazebo>
-    <!-- Femur Link -->
-    <gazebo reference="femur_link">
+    <gazebo reference="coxa_link_1">
+      <mu1>0.2</mu1>
+      <mu2>0.2</mu2>
+      <material>Gazebo/Blue</material>
+    </gazebo>
+    <gazebo reference="coxa_link_2">
+      <mu1>0.2</mu1>
+      <mu2>0.2</mu2>
+      <material>Gazebo/Blue</material>
+    </gazebo>
+    <gazebo reference="coxa_link_3">
+      <mu1>0.2</mu1>
+      <mu2>0.2</mu2>
+      <material>Gazebo/Blue</material>
+    </gazebo>
+    <gazebo reference="coxa_link_4">
+      <mu1>0.2</mu1>
+      <mu2>0.2</mu2>
+      <material>Gazebo/Blue</material>
+    </gazebo>
+    <gazebo reference="coxa_link_5">
+      <mu1>0.2</mu1>
+      <mu2>0.2</mu2>
+      <material>Gazebo/Blue</material>
+    </gazebo>
+    <!-- Femur Links -->
+    <gazebo reference="femur_link_0">
       <mu1>0.2</mu1>
       <mu2>0.2</mu2>
       <material>Gazebo/Orange</material>
     </gazebo>
-    <!-- Tibia Link -->
-    <gazebo reference="tibia_link">
+    <gazebo reference="femur_link_1">
+      <mu1>0.2</mu1>
+      <mu2>0.2</mu2>
+      <material>Gazebo/Orange</material>
+    </gazebo>
+    <gazebo reference="femur_link_2">
+      <mu1>0.2</mu1>
+      <mu2>0.2</mu2>
+      <material>Gazebo/Orange</material>
+    </gazebo>
+    <gazebo reference="femur_link_3">
+      <mu1>0.2</mu1>
+      <mu2>0.2</mu2>
+      <material>Gazebo/Orange</material>
+    </gazebo>
+    <gazebo reference="femur_link_4">
+      <mu1>0.2</mu1>
+      <mu2>0.2</mu2>
+      <material>Gazebo/Orange</material>
+    </gazebo>
+    <gazebo reference="femur_link_5">
+      <mu1>0.2</mu1>
+      <mu2>0.2</mu2>
+      <material>Gazebo/Orange</material>
+    </gazebo>
+    <!-- Tibia Links -->
+    <gazebo reference="tibia_link_0">
+      <mu1>0.2</mu1>
+      <mu2>0.2</mu2>
+      <material>Gazebo/Black</material>
+    </gazebo>
+    <gazebo reference="tibia_link_1">
+      <mu1>0.2</mu1>
+      <mu2>0.2</mu2>
+      <material>Gazebo/Black</material>
+    </gazebo>
+    <gazebo reference="tibia_link_2">
+      <mu1>0.2</mu1>
+      <mu2>0.2</mu2>
+      <material>Gazebo/Black</material>
+    </gazebo>
+    <gazebo reference="tibia_link_3">
+      <mu1>0.2</mu1>
+      <mu2>0.2</mu2>
+      <material>Gazebo/Black</material>
+    </gazebo>
+    <gazebo reference="tibia_link_4">
+      <mu1>0.2</mu1>
+      <mu2>0.2</mu2>
+      <material>Gazebo/Black</material>
+    </gazebo>
+    <gazebo reference="tibia_link_5">
       <mu1>0.2</mu1>
       <mu2>0.2</mu2>

File: silver/description/robot_core.xacro (robot description, xacro)
@@ -89,5 +89,4 @@
     </link>
 <!-- TIBIA JOINT AND LINK -->
-<!-- Simulate the 4 bar mechanism is not possible with urfd. Must look into transmission/mapping between motor angle and joint angle -->
     <joint name="tibia_joint" type="revolute">
         <origin xyz="${tibia_joint_Ox} ${tibia_joint_Oy} ${tibia_joint_Oz}" rpy="0.0 0.0 0.0"/>
@@ -117,10 +116,10 @@
     </link>
 <!-- FOOT JOINT (FIXED) AND LINK -->
-    <joint name="foot_joint" type="fixed">
+    <!--joint name="foot_joint" type="fixed">
         <origin xyz="${foot_joint_Ox} 0.0 0.0" rpy="0.0 0.0 ${foot_joint_Rz}"/>
         <parent link="tibia_link"/>
         <child link="foot_link"/>
-    </joint>
-     <link name="foot_link">
+    </joint-->
+     <!--link name="foot_link">
         <visual>
             <origin xyz="${foot_link_Ox} 0.0 0.0" rpy="0.0 0.0 0.0"/>
@@ -139,4 +138,4 @@
             <origin xyz="${foot_link_Ox} 0.0 0.0" rpy="0.0 0.0 0.0"/>
         </xacro:inertial_box>
-    </link>
+    </link-->
 </robot>

File: silver/description/ros2_control.xacro (robot description, xacro)
@@ -10,4 +10,5 @@
             <hardware>
                 <plugin>dynamixel_hardware/DynamixelHardware</plugin>
+                <!--plugin>silver_dynamixel_hardware/SilverDynamixelHardware</plugin-->
                 <param name="usb_port">/dev/ttyUSB0</param>
                 <param name="baud_rate">57600</param>
@@ -20,4 +21,8 @@
                 <param name="max">3.14</param>
             </command_interface>
+            <command_interface name="velocity"/>
+            <xacro:if value="$(arg sim_mode)">
+                <command_interface name="effort"/>
+            </xacro:if>
             <state_interface name="position"/>
             <state_interface name="velocity"/>
@@ -30,4 +35,8 @@
                 <param name="max">3.14</param>
             </command_interface>
+            <command_interface name="velocity"/>
+            <xacro:if value="$(arg sim_mode)">
+                <command_interface name="effort"/>
+            </xacro:if>
             <state_interface name="position"/>
             <state_interface name="velocity"/>
@@ -40,8 +49,36 @@
                 <param name="max">3.14</param>
             </command_interface>
+            <command_interface name="velocity"/>
+            <xacro:if value="$(arg sim_mode)">
+                <command_interface name="effort"/>
+            </xacro:if>
             <state_interface name="position"/>
             <state_interface name="velocity"/>
             <state_interface name="effort"/>
         </joint>
+        <!---transmission name="coxa_transmission">
+            <plugin>transmission_interface/SimpleTransmission</plugin>
+            <actuator name="coxa_motor" role="coxa_motor"/>
+            <joint name="coxa_joint" role="coxa_joint">
+                <mechanical_reduction>1.0</mechanical_reduction>
+                <offset>0.0</offset>
+            </joint>
+        </transmission>
+        <transmission name="femur_transmission">
+            <plugin>transmission_interface/SimpleTransmission</plugin>
+            <actuator name="femur_motor" role="femur_motor"/>
+            <joint name="femur_joint" role="femur_joint">
+                <mechanical_reduction>1.0</mechanical_reduction>
+                <offset>0.0</offset>
+            </joint>
+        </transmission>
+        <transmission name="tibia_transmssion">
+            <plugin>transmission_interface/SimpleTransmission</plugin>
+            <actuator name="tibia_motor" role="tibia_motor"/>
+            <joint name="tibia_joint" role="tibia_joint">
+                <mechanical_reduction>4.0</mechanical_reduction>
+                <offset>0.0</offset>
+            </joint>
+        </transmission-->
     </ros2_control>
 </robot>

File: silver/description/silver_constants.xacro (robot description, xacro)
@@ -5,10 +5,10 @@
     <xacro:property name="body_link_height" value="1.0" /> <!-- m -->
     <xacro:property name="body_link_x_dim" value="0.8" /> <!-- m -->
-    <xacro:property name="body_link_y_dim" value="0.5" /> <!-- m -->
+    <xacro:property name="body_link_y_dim" value="0.6" /> <!-- m -->
     <xacro:property name="body_link_z_dim" value="0.3" /> <!-- m -->
     <xacro:property name="coxa_link_mass" value="0.5" /> <!-- Kg -->
-    <xacro:property name="coxa_joint_Ox" value="0.35" /> <!-- m -->
-    <xacro:property name="coxa_joint_Oy" value="0.2" /> <!-- m -->
-    <xacro:property name="coxa_joint_Oz" value="-0.15" /> <!-- m -->
+    <xacro:property name="coxa_joint_Ox" value="0.0" /> <!-- m -->
+    <xacro:property name="coxa_joint_Oy" value="0.0" /> <!-- m -->
+    <xacro:property name="coxa_joint_Oz" value="0.0" /> <!-- m -->
     <xacro:property name="coxa_link_Ox" value="0.03" /> <!-- m -->
     <xacro:property name="coxa_link_Oy" value="0.05" /> <!-- m -->
@@ -42,5 +42,5 @@
     <xacro:property name="foot_joint_Oy" value="0.0" /> <!-- m -->
     <xacro:property name="foot_joint_Oz" value="0.0" /> <!-- m -->
-    <xacro:property name="foot_joint_Rz" value="-0.785" /> <!-- m -->
+    <xacro:property name="foot_joint_Rz" value="-0.785" /> <!-- rad -->
     <xacro:property name="foot_link_Ox" value="0.01" /> <!-- m -->
     <xacro:property name="foot_link_Oy" value="0.0" /> <!-- m -->
