Commit message: Add files via upload

File: silver/description/gazebo_control.xacro (robot description, xacro)
@@ -8,108 +8,3 @@
       </plugin>
     </gazebo>
-     <!-- Body Link -->
-    <gazebo reference="body_link">
-      <mu1>0.2</mu1>
-      <mu2>0.2</mu2>
-      <material>Gazebo/Blue</material>
-    </gazebo>
-    <!-- Coxa Links -->
-    <gazebo reference="coxa_link_0">
-      <mu1>0.2</mu1>
-      <mu2>0.2</mu2>
-      <material>Gazebo/Blue</material>
-    </gazebo>
-    <gazebo reference="coxa_link_1">
-      <mu1>0.2</mu1>
-      <mu2>0.2</mu2>
-      <material>Gazebo/Blue</material>
-    </gazebo>
-    <gazebo reference="coxa_link_2">
-      <mu1>0.2</mu1>
-      <mu2>0.2</mu2>
-      <material>Gazebo/Blue</material>
-    </gazebo>
-    <gazebo reference="coxa_link_3">
-      <mu1>0.2</mu1>
-      <mu2>0.2</mu2>
-      <material>Gazebo/Blue</material>
-    </gazebo>
-    <gazebo reference="coxa_link_4">
-      <mu1>0.2</mu1>
-      <mu2>0.2</mu2>
-      <material>Gazebo/Blue</material>
-    </gazebo>
-    <gazebo reference="coxa_link_5">
-      <mu1>0.2</mu1>
-      <mu2>0.2</mu2>
-      <material>Gazebo/Blue</material>
-    </gazebo>
-    <!-- Femur Links -->
-    <gazebo reference="femur_link_0">
-      <mu1>0.2</mu1>
-      <mu2>0.2</mu2>
-      <material>Gazebo/Orange</material>
-    </gazebo>
-    <gazebo reference="femur_link_1">
-      <mu1>0.2</mu1>
-      <mu2>0.2</mu2>
-      <material>Gazebo/Orange</material>
-    </gazebo>
-    <gazebo reference="femur_link_2">
-      <mu1>0.2</mu1>
-      <mu2>0.2</mu2>
-      <material>Gazebo/Orange</material>
-    </gazebo>
-    <gazebo reference="femur_link_3">
-      <mu1>0.2</mu1>
-      <mu2>0.2</mu2>
-      <material>Gazebo/Orange</material>
-    </gazebo>
-    <gazebo reference="femur_link_4">
-      <mu1>0.2</mu1>
-      <mu2>0.2</mu2>
-      <material>Gazebo/Orange</material>
-    </gazebo>
-    <gazebo reference="femur_link_5">
-      <mu1>0.2</mu1>
-      <mu2>0.2</mu2>
-      <material>Gazebo/Orange</material>
-    </gazebo>
-    <!-- Tibia Links -->
-    <gazebo reference="tibia_link_0">
-      <mu1>0.2</mu1>
-      <mu2>0.2</mu2>
-      <material>Gazebo/Black</material>
-    </gazebo>
-    <gazebo reference="tibia_link_1">
-      <mu1>0.2</mu1>
-      <mu2>0.2</mu2>
-      <material>Gazebo/Black</material>
-    </gazebo>
-    <gazebo reference="tibia_link_2">
-      <mu1>0.2</mu1>
-      <mu2>0.2</mu2>
-      <material>Gazebo/Black</material>
-    </gazebo>
-    <gazebo reference="tibia_link_3">
-      <mu1>0.2</mu1>
-      <mu2>0.2</mu2>
-      <material>Gazebo/Black</material>
-    </gazebo>
-    <gazebo reference="tibia_link_4">
-      <mu1>0.2</mu1>
-      <mu2>0.2</mu2>
-      <material>Gazebo/Black</material>
-    </gazebo>
-    <gazebo reference="tibia_link_5">
-      <mu1>0.2</mu1>
-      <mu2>0.2</mu2>
-      <material>Gazebo/Black</material>
-    </gazebo>
-    <!-- Foot Link -->
-    <gazebo reference="foot_link">
-      <mu1>0.2</mu1>
-      <mu2>0.2</mu2>
-      <material>Gazebo/Orange</material>
-    </gazebo>
 </robot>

File: silver/description/ros2_control_leg.xacro (robot description, xacro)
@@ -3,42 +3,93 @@
     <xacro:macro name="leg_control" params="suffix">
         <joint name="coxa_joint_${suffix}">
-        <param name="id">${suffix*3 + 0}</param>
-            <command_interface name="position">
+            <param name="id">${suffix*3 + 0}</param>
+            <param name="pos_kp">5000</param>
+            <param name="pos_ki">1</param>
+            <param name="pos_kd">3</param>
+            <param name="pos_max_integral_error">10000</param>
+            <command_interface name="position_pid">
+            <!--command_interface name="position"-->
                 <param name="min">-3.14</param>
                 <param name="max">3.14</param>
             </command_interface>
-            <command_interface name="velocity"/>
+            <command_interface name="velocity">
+                <!--param name="min">-1.0</param>
+                <param name="max">1.0</param-->
+            </command_interface>
             <xacro:if value="$(arg sim_mode)">
                 <command_interface name="effort"/>
             </xacro:if>
-            <state_interface name="position"/>
+            <!--state_interface name="position"/-->
+            <!--SET INITIAL POSITION, note that this will not reset when gazebo world is restarted-->
+            <state_interface name="position">
+                <xacro:if value="${suffix==0}">
+                    <param name="initial_value">0.75</param>
+                </xacro:if>
+                <xacro:if value="${suffix==1}">
+                    <param name="initial_value">0.0</param>
+                </xacro:if>
+                <xacro:if value="${suffix==2}">
+                    <param name="initial_value">-0.75</param>
+                </xacro:if>
+                <xacro:if value="${suffix==3}">
+                    <param name="initial_value">-0.75</param>
+                </xacro:if>
+                <xacro:if value="${suffix==4}">
+                    <param name="initial_value">0.0</param>
+                </xacro:if>
+                <xacro:if value="${suffix==5}">
+                    <param name="initial_value">0.75</param>
+                </xacro:if>
+            </state_interface>
             <state_interface name="velocity"/>
             <state_interface name="effort"/>
         </joint>
         <joint name="femur_joint_${suffix}">
-        <param name="id">${suffix*3 + 1}</param>
-            <command_interface name="position">
+            <param name="id">${suffix*3 + 1}</param>
+            <param name="pos_kp">5000</param>
+            <param name="pos_ki">1</param>
+            <param name="pos_kd">3</param>
+            <param name="pos_max_integral_error">10000</param>
+            <command_interface name="position_pid">
+            <!--command_interface name="position"-->
                 <param name="min">-3.14</param>
                 <param name="max">3.14</param>
             </command_interface>
-            <command_interface name="velocity"/>
+            <command_interface name="velocity">
+                <!--param name="min">-1.0</param>
+                <param name="max">1.0</param-->
+            </command_interface>
             <xacro:if value="$(arg sim_mode)">
                 <command_interface name="effort"/>
             </xacro:if>
-            <state_interface name="position"/>
+            <!--state_interface name="position"/-->
+            <state_interface name="position">
+                <param name="initial_value">0.8</param>
+            </state_interface>
             <state_interface name="velocity"/>
             <state_interface name="effort"/>
         </joint>
         <joint name="tibia_joint_${suffix}">
-        <param name="id">${suffix*3 + 2}</param>
-            <command_interface name="position">
+            <param name="id">${suffix*3 + 2}</param>
+            <param name="pos_kp">5000</param>
+            <param name="pos_ki">1</param>
+            <param name="pos_kd">3</param>
+            <param name="pos_max_integral_error">10000</param>
+            <command_interface name="position_pid">
+            <!--command_interface name="position"-->
                 <param name="min">-3.14</param>
                 <param name="max">3.14</param>
             </command_interface>
-            <command_interface name="velocity"/>
+            <command_interface name="velocity">
+                <!--param name="min">-1.0</param>
+                <param name="max">1.0</param-->
+            </command_interface>
             <xacro:if value="$(arg sim_mode)">
                 <command_interface name="effort"/>
             </xacro:if>
-            <state_interface name="position"/>
+            <!--state_interface name="position"/-->
+            <state_interface name="position">
+                <param name="initial_value">2.3</param>
+            </state_interface>
             <state_interface name="velocity"/>
             <state_interface name="effort"/>

File: silver/description/silver.xacro (robot description, xacro)
@@ -17,11 +17,10 @@
     <!-- Import Rviz colors -->
     <xacro:include filename="colors_rviz.xacro"/>
-    <!-- WORLD LINK -->
-    <link name = "world"></link>
+    <!-- BASE LINK -->
+    <link name = "base_link"></link>
     <!-- BODY JOINT AND LINK -->
-    <!-- BODY joint will be made non fixed when the whole robot is ready-->
     <joint name="body_joint" type="fixed">
-        <origin xyz="0.0 0.0 ${body_link_height}" rpy="0.0 0.0 0.0"/>
-        <parent link="world"/>
+        <origin xyz="0.0 0.0 0.4" rpy="0.0 0.0 0.0"/>
+        <parent link="base_link"/>
         <child link="body_link"/>
     </joint>
@@ -44,4 +43,10 @@
         </xacro:inertial_box>
     </link>
+    <!-- Body Link -->
+    <gazebo reference="body_link">
+      <!--mu1>50.0</mu1>
+      <mu2>50.0</mu2-->
+      <material>Gazebo/Blue</material>
+    </gazebo>
     <xacro:leg suffix="0" reflect="1" side='right' Ox="0.275" Oy="-0.2" Oz="-0.15"/>
     <xacro:leg suffix="1" reflect="1" side='right' Ox="0.0" Oy="-0.2" Oz="-0.15"/>

File: silver/description/silver_constants.xacro (robot description, xacro)
@@ -2,10 +2,10 @@
 <robot xmlns:xacro="http://www.ros.org/wiki/xacro" >
     <!-- Constant parameters -->
-    <xacro:property name="body_link_mass" value="2.0" /> <!-- Kg -->
+    <xacro:property name="body_link_mass" value="140.0" /> <!-- Kg -->
     <xacro:property name="body_link_height" value="1.0" /> <!-- m -->
     <xacro:property name="body_link_x_dim" value="0.55" /> <!-- m -->
     <xacro:property name="body_link_y_dim" value="0.4" /> <!-- m -->
     <xacro:property name="body_link_z_dim" value="0.3" /> <!-- m -->
-    <xacro:property name="coxa_link_mass" value="0.5" /> <!-- Kg -->
+    <xacro:property name="coxa_link_mass" value="0.301" /> <!-- Kg -->
     <xacro:property name="coxa_joint_Ox" value="0.0" /> <!-- m -->
     <xacro:property name="coxa_joint_Oy" value="0.0" /> <!-- m -->
@@ -17,5 +17,5 @@
     <xacro:property name="coxa_link_length" value="0.1" /> <!-- m -->
     <xacro:property name="coxa_link_radius" value="0.05" /> <!-- m -->
-    <xacro:property name="femur_link_mass" value="0.5" /> <!-- Kg -->
+    <xacro:property name="femur_link_mass" value="0.501" /> <!-- Kg -->
     <xacro:property name="femur_joint_Ox" value="0.07" /> <!-- m -->
     <xacro:property name="femur_joint_Oy" value="-0.05" /> <!-- m -->
@@ -24,9 +24,9 @@
     <xacro:property name="femur_link_Ox" value="0.0" /> <!-- m -->
     <xacro:property name="femur_link_Oy" value="-0.15" /> <!-- m -->
-    <xacro:property name="femur_link_Oz" value="-0.01" /> <!-- m -->
+    <xacro:property name="femur_link_Oz" value="-0.03" /> <!-- m -->
     <xacro:property name="femur_link_dx" value="0.03" /> <!-- m -->
     <xacro:property name="femur_link_dy" value="0.3" /> <!-- m -->
     <xacro:property name="femur_link_dz" value="0.01" /> <!-- m -->
-    <xacro:property name="tibia_link_mass" value="0.5" /> <!-- Kg -->
+    <xacro:property name="tibia_link_mass" value="0.401" /> <!-- Kg -->
     <xacro:property name="tibia_joint_Ox" value="0.0" /> <!-- m -->
     <xacro:property name="tibia_joint_Oy" value="-0.3" /> <!-- m -->
@@ -37,16 +37,14 @@
     <xacro:property name="tibia_link_Oz" value="0.0" /> <!-- m -->
     <xacro:property name="tibia_link_dx" value="0.03" /> <!-- m -->
-    <xacro:property name="tibia_link_dy" value="-0.32" /> <!-- m -->
+    <xacro:property name="tibia_link_dy" value="-0.27" /> <!-- m -->
     <xacro:property name="tibia_link_dz" value="0.01" /> <!-- m -->
-    <xacro:property name="foot_link_mass" value="0.1" /> <!-- Kg -->
-    <xacro:property name="foot_joint_Ox" value="0.3" /> <!-- m -->
-    <xacro:property name="foot_joint_Oy" value="0.0" /> <!-- m -->
+    <xacro:property name="foot_mass" value="0.001" /> <!-- Kg -->
+    <xacro:property name="foot_radius" value="0.025" /> <!-- m -->
+    <xacro:property name="foot_joint_Ox" value="0.0" /> <!-- m -->
+    <xacro:property name="foot_joint_Oy" value="-0.295" /> <!-- m -->
     <xacro:property name="foot_joint_Oz" value="0.0" /> <!-- m -->
-    <xacro:property name="foot_joint_Rz" value="-0.785" /> <!-- rad -->
-    <xacro:property name="foot_link_Ox" value="0.01" /> <!-- m -->
+    <xacro:property name="foot_joint_Rz" value="0.0" /> <!-- rad -->
+    <xacro:property name="foot_link_Ox" value="0.0" /> <!-- m -->
     <xacro:property name="foot_link_Oy" value="0.0" /> <!-- m -->
     <xacro:property name="foot_link_Oz" value="0.0" /> <!-- m -->
-    <xacro:property name="foot_link_dx" value="0.05" /> <!-- m -->
-    <xacro:property name="foot_link_dy" value="0.01" /> <!-- m -->
-    <xacro:property name="foot_link_dz" value="0.01" /> <!-- m -->
 </robot>

File: silver/description/silver_constants_new.xacro (robot description, xacro)
@@ -1,5 +1,5 @@
 <?xml version="1.0"?>
 <robot xmlns:xacro="http://www.ros.org/wiki/xacro" >
-    <!-- Constant parameters -->
+    <!-- Constant parameters for new leg (all motors in one canister)-->
     <xacro:property name="body_link_mass" value="2.0" /> <!-- Kg -->
     <xacro:property name="body_link_height" value="1.0" /> <!-- m -->

File: silver/description/silver_leg.xacro (robot description, xacro)
@@ -12,7 +12,7 @@
             <parent link="body_link"/>
             <child link="coxa_link_${suffix}"/>
-            <limit effort="100" velocity="100.0" lower="-3.14" upper="3.14" />
+            <limit effort="250.0" velocity="10.0" lower="-3.14" upper="3.14" />
             <axis xyz="0 0 1"/>
-            <dynamics damping="0.7"/>
+            <!--dynamics damping="10.0" friction="10.0"/-->
         </joint>
         <link name="coxa_link_${suffix}">
@@ -34,4 +34,11 @@
             </xacro:inertial_cylinder>
         </link>
+        <gazebo reference="coxa_link_${suffix}">
+            <!--mu1>50.0</mu1>
+            <mu2>50.0</mu2>
+            <kp>1e13</kp>
+            <kd>1e15</kd-->
+            <material>Gazebo/Blue</material>
+        </gazebo>
         <!-- FEMUR JOINT AND LINK-->
         <joint name="femur_joint_${suffix}" type="revolute">
@@ -39,7 +46,7 @@
             <parent link="coxa_link_${suffix}"/>
             <child link="femur_link_${suffix}"/>
-            <limit effort="100" velocity="100.0" lower="-3.14" upper="3.14" />
+            <limit effort="250.0" velocity="10.0" lower="-3.14" upper="3.14" />
             <axis xyz="0 0 1"/>
-            <dynamics damping="0.7"/>
+            <!--dynamics damping="10.0" friction="10.0"/-->
         </joint>
         <link name="femur_link_${suffix}">
@@ -61,4 +68,11 @@
             </xacro:inertial_box>
         </link>
+        <gazebo reference="femur_link_${suffix}">
+            <!--mu1>50.0</mu1>
+            <mu2>50.0</mu2>
+            <kp>1e13</kp>
+            <kd>1e15</kd-->
+            <material>Gazebo/Orange</material>
+        </gazebo>
         <!-- TIBIA JOINT AND LINK -->
         <joint name="tibia_joint_${suffix}" type="revolute">
@@ -66,7 +80,7 @@
             <parent link="femur_link_${suffix}"/>
             <child link="tibia_link_${suffix}"/>
-            <limit effort="100" velocity="100.0" lower="-3.14" upper="3.14" />
+            <limit effort="250.0" velocity="10.0" lower="-3.14" upper="3.14" />
             <axis xyz="0 0 1"/>
-            <dynamics damping="0.7"/>
+            <!--dynamics damping="10.0" friction="10.0"/-->
         </joint>
         <link name="tibia_link_${suffix}">
@@ -88,4 +102,47 @@
             </xacro:inertial_box>
         </link>
+        <gazebo reference="tibia_link_${suffix}">
+            <!--mu1>2000.0</mu1>
+            <mu2>2000.0</mu2>
+            <kp>0.1</kp>
+            <kd>0.1</kd-->
+            <material>Gazebo/Black</material>
+        </gazebo>
+        <!-- FOOT JOINT AND LINK -->
+        <joint name="foot_joint_${suffix}" type="fixed">
+            <origin xyz="${foot_joint_Ox} ${foot_joint_Oy} ${foot_joint_Oz}" rpy="0.0 0.0 0.0"/>
+            <parent link="tibia_link_${suffix}"/>
+            <child link="foot_link_${suffix}"/>
+        </joint>
+        <link name="foot_link_${suffix}">
+            <visual>
+                <origin xyz="${foot_link_Ox} ${foot_link_Oy} ${foot_link_Oz}" rpy="0.0 0.0 0.0"/>
+                <geometry>
+                    <sphere radius="${foot_radius}"/>
+                    <!--box size="0.1 0.05 0.05"/-->
+                </geometry>
+                <material name="white"/>
+            </visual>
+            <collision>
+                <origin xyz="${foot_link_Ox} ${foot_link_Oy} ${foot_link_Oz}" rpy="0.0 0.0 0.0"/>
+                <geometry>
+                    <sphere radius="${foot_radius}"/>
+                    <!--box size="0.1 0.05 0.05"/-->
+                </geometry>
+            </collision>
+            <xacro:inertial_sphere mass="${foot_mass}" radius="${foot_radius}">
+                <origin xyz="${foot_link_Ox} ${foot_link_Oy} ${foot_link_Oz}" rpy="0.0 0.0 0.0"/>
+            </xacro:inertial_sphere>
+            <!--xacro:inertial_box mass="${foot_mass}" x="0.1" y="0.05" z="0.05">
+                <origin xyz="${foot_link_Ox} ${foot_link_Oy} ${foot_link_Oz}" rpy="0.0 0.0 0.0"/>
+            </xacro:inertial_box-->
+        </link>
+        <gazebo reference="foot_link_${suffix}">
+            <!--mu1>2000.0</mu1>
+            <mu2>2000.0</mu2>
+            <kp>1e3</kp>
+            <kd>1e5</kd-->
+            <material>Gazebo/White</material>
+        </gazebo>
     </xacro:macro>
 </robot>

File: silver/description/silver_leg_new.xacro (robot description, xacro)
@@ -7,7 +7,7 @@
                 <parent link="body_link"/>
                 <child link="coxa_link_${suffix}"/>
-                <limit effort="100" velocity="100.0" lower="-3.14" upper="3.14" />
+                <limit effort="3" velocity="100.0" lower="-3.14" upper="3.14" />
                 <axis xyz="0 0 1"/>
-                <dynamics damping="0.7"/>
+                <!--dynamics damping="0.7"/-->
         </joint>
         <link name="coxa_link_${suffix}">
@@ -34,7 +34,7 @@
             <parent link="coxa_link_${suffix}"/>
             <child link="femur_link_${suffix}"/>
-            <limit effort="100" velocity="100.0" lower="-3.14" upper="3.14" />
+            <limit effort="3" velocity="100.0" lower="-3.14" upper="3.14" />
             <axis xyz="0 0 ${reflect}"/>
-            <dynamics damping="0.7"/>
+            <!--dynamics damping="0.7"/-->
         </joint>
         <link name="femur_link_${suffix}">
@@ -61,7 +61,7 @@
             <parent link="femur_link_${suffix}"/>
             <child link="tibia_link_${suffix}"/>
-            <limit effort="100" velocity="100.0" lower="-3.14" upper="3.14" />
+            <limit effort="3" velocity="100.0" lower="-3.14" upper="3.14" />
             <axis xyz="0 0 ${reflect}"/>
-            <dynamics damping="0.7"/>
+            <!--dynamics damping="0.7"/-->
         </joint>
         <link name="tibia_link_${suffix}">
