Commit message: Add files via upload

File: silver/description/silver.xacro (robot description, xacro)
@@ -26,4 +26,11 @@
     </joint>
     <link name="body_link">
+        <!--visual>
+            <origin xyz="1.0 0.0 0.0" rpy="1.57 0.0 1.57"/>
+            <geometry>
+                <mesh filename="package://silver/meshes/body_lowresolution.STL" scale="0.005 0.005 0.005"/>
+            </geometry>
+            <material name="blue"/>
+        </visual-->
         <visual>
             <origin xyz="0.0 0.0 0.0" rpy="0.0 0.0 0.0"/>
